File: kicad/hours.sch (KiCad schematic (older format))
At the start: 0 parts

Commit message: hours section
Parts:
- added AFF5, AFF6: 7SEGMENTS, symbol 7SEGMENTS
- added R8: 1K, symbol R
- added RP5, RP6: 1K, symbol R_PACK8
- added U14, U15: 74LS90, symbol 74LS90
- added U16, U17: 74LS47, symbol 74LS47
Connections:
- new net: U15.1 (CP1..3), U15.12 (Q0), U17.7 (A)
- new net: U14.1 (CP1..3), U15.11 (Q3), U17.6 (D)
- new net: U14.2 (R0(1)), U15.2 (R0(1)), U15.8 (Q2), U17.2 (C)
- new net: U14.3 (R0(2)), U14.8 (Q2), U15.3 (R0(2)), U16.1 (B)
- new net: U15.9 (Q1), U17.1 (B)
- new net: RP5.4 (P4), U16.10 (d)
- new net: RP5.3 (P3), U16.11 (c)
- new net: RP5.2 (P2), U16.12 (b)
- new net: RP5.1 (P1), U16.13 (a)
- new net: RP5.7 (P7), U16.14 (g)
- new net: RP5.6 (P6), U16.15 (f)
- new net: U14.11 (Q3), U16.2 (C)
- new net: U14.9 (Q1), U16.7 (A)
- new net: RP5.5 (P5), U16.9 (e)
- new net: RP6.4 (P4), U17.10 (d)
- new net: RP6.3 (P3), U17.11 (c)
- new net: RP6.2 (P2), U17.12 (b)
- new net: RP6.1 (P1), U17.13 (a)
- new net: RP6.7 (P7), U17.14 (g)
- new net: RP6.6 (P6), U17.15 (f)
- new net: RP6.5 (P5), U17.9 (e)
- new net: AFF5.1 (e), RP5.12 (R5)
- new net: AFF5.10 (g), RP5.10 (R7)
- new net: AFF5.2 (d), RP5.13 (R4)
- new net: AFF5.4 (c), RP5.14 (R3)
- new net: AFF5.6 (b), RP5.15 (R2)
- new net: AFF5.7 (a), RP5.16 (R1)
- new net: AFF5.9 (f), RP5.11 (R6)
- new net: AFF6.1 (e), RP6.12 (R5)
- new net: AFF6.10 (g), RP6.10 (R7)
- new net: AFF6.2 (d), RP6.13 (R4)
- new net: AFF6.4 (c), RP6.14 (R3)
- new net: AFF6.6 (b), RP6.15 (R2)
- new net: AFF6.7 (a), RP6.16 (R1)
- new net: AFF6.9 (f), RP6.11 (R6)
- new net: R8.2, U14.14 (CP0)
- new net +5V: AFF5.3 (C.A.), AFF6.3 (C.A.), R8.1
- new net GND: U14.6 (R9(1)), U15.6 (R9(1)), U16.6 (D), U16.8 (GND), U17.8 (GND)
- new net HOUR_CLK: U15.14 (CP0)
- new net VCC: U14.5 (VCC), U15.5 (VCC), U16.16 (VCC), U17.16 (VCC)
