File: kicad/minutes.sch (KiCad schematic (older format))
At the start: 0 parts

Commit message: minute segment
Parts:
- added AFF? (x2): 7SEGMENTS, symbol 7SEGMENTS
- added RP? (x2): 1K, symbol R_PACK8
- added U?: 74LS90, symbol 74LS90
- added U?: 74LS92, symbol 74LS92
- added U? (x2): 74LS47, symbol 74LS47
Connections:
- new net: U?.1 (CP1..3), U?.12 (Q0), U?.7 (A) (x2)
- new net: U?.11 (Q3), U?.14 (CP0), U?.6 (D)
- new net: U?.2 (C), U?.8 (Q2)
- new net: U?.1 (B), U?.9 (Q1)
- new net: U?.1 (B), U?.11 (Q1)
- new net: RP?.4 (P4), U?.10 (d) (x2)
- new net: RP?.3 (P3), U?.11 (c) (x2)
- new net: RP?.2 (P2), U?.12 (b) (x2)
- new net: RP?.1 (P1), U?.13 (a) (x2)
- new net: RP?.7 (P7), U?.14 (g) (x2)
- new net: RP?.6 (P6), U?.15 (f) (x2)
- new net: RP?.5 (P5), U?.9 (e) (x2)
- new net: AFF?.1 (e), RP?.12 (R5) (x2)
- new net: AFF?.10 (g), RP?.10 (R7) (x2)
- new net: AFF?.2 (d), RP?.13 (R4) (x2)
- new net: AFF?.4 (c), RP?.14 (R3) (x2)
- new net: AFF?.6 (b), RP?.15 (R2) (x2)
- new net: AFF?.7 (a), RP?.16 (R1) (x2)
- new net: AFF?.9 (f), RP?.11 (R6) (x2)
- new net +5V: AFF?.3 (C.A.)
- new net GND: U?.2 (R0(1)), U?.6 (D), U?.6 (R0(1)), U?.8 (GND), U?.8 (GND)
- new net HOUR_PULSE: U?.2 (C), U?.9 (Q2)
- new net MINUTE_CLK: U?.14 (CP0)
- new net VCC: U?.16 (VCC), U?.16 (VCC), U?.5 (VCC), U?.5 (VCC)
Changed lines of the file:
@@
 $Descr A4 11693 8268
 encoding utf-8
-Sheet 1 5
+Sheet 4 5
 Title ""
 Date ""
@@
 Comment4 ""
 $EndDescr
+$Comp
+L 74LS90 U?
+U 1 1 5F410FEF
+P 3250 4650
+F 0 "U?" H 3350 4650 50  0000 C CNN
+F 1 "74LS90" H 3450 4450 50  0000 C CNN
+F 2 "" H 3250 4650 50  0000 C CNN
+F 3 "" H 3250 4650 50  0000 C CNN
+	1    3250 4650
+	1    0    0    -1
+$EndComp
+$Comp
+L 74LS92 U?
+U 1 1 5F410FF6
+P 3250 2300
+F 0 "U?" H 3350 2300 50  0000 C CNN
+F 1 "74LS92" H 3450 2100 50  0000 C CNN
+F 2 "" H 3250 2300 50  0000 C CNN
+F 3 "" H 3250 2300 50  0000 C CNN
+	1    3250 2300
+	1    0    0    -1
+$EndComp
+$Comp
+L GND #PWR?
+U 1 1 5F410FFD
+P 2550 5150
+F 0 "#PWR?" H 2550 4900 50  0001 C CNN
+F 1 "GND" H 2550 5000 50  0000 C CNN
+F 2 "" H 2550 5150 50  0000 C CNN
+F 3 "" H 2550 5150 50  0000 C CNN
+	1    2550 5150
+	1    0    0    -1
+$EndComp
+Wire Wire Line
+	2550 4600 2550 5150
+$Comp
+L GND #PWR?
+U 1 1 5F411004
+P 2550 2850
+F 0 "#PWR?" H 2550 2600 50  0001 C CNN
+F 1 "GND" H 2550 2700 50  0000 C CNN
+F 2 "" H 2550 2850 50  0000 C CNN
+F 3 "" H 2550 2850 50  0000 C CNN
+	1    2550 2850
+	1    0    0    -1
+$EndComp
+Wire Wire Line
+	2550 2250 2550 2850
+Wire Wire Line
+	2550 4350 2250 4350
+Wire Wire Line
+	2550 4450 2400 4450
+Wire Wire Line
+	2400 4450 2400 4100
+Wire Wire Line
+	2400 4100 4000 4100
+Wire Wire Line
+	4000 4100 4000 4350
+Wire Wire Line
+	4000 4650 4750 4650
+Wire Wire Line
+	4250 4650 4250 3950
+Wire Wire Line
+	4250 3950 2300 3950
+Wire Wire Line
+	2300 3950 2300 2000
+Wire Wire Line
+	2300 2000 2550 2000
+Wire Wire Line
+	4000 2000 4000 1700
+Wire Wire Line
+	4000 1700 2550 1700
+Wire Wire Line
+	2550 1700 2550 2100
+Wire Wire Line
+	4150 2550 4150 2200
+Wire Wire Line
+	4000 2200 4750 2200
+$Comp
+L 74LS47 U?
+U 1 1 5F41101C
+P 5450 2350
+F 0 "U?" H 5450 2450 50  0000 C CNN
+F 1 "74LS47" H 5450 2250 50  0000 C CNN
+F 2 "" H 5450 2350 50  0000 C CNN
+F 3 "" H 5450 2350 50  0000 C CNN
+	1    5450 2350
+	1    0    0    -1
+$EndComp
+$Comp
+L 74LS47 U?
+U 1 1 5F411023
+P 5450 4700
+F 0 "U?" H 5450 4800 50  0000 C CNN
+F 1 "74LS47" H 5450 4600 50  0000 C CNN
+F 2 "" H 5450 4700 50  0000 C CNN
+F 3 "" H 5450 4700 50  0000 C CNN
+	1    5450 4700
+	1    0    0    -1
+$EndComp
+Wire Wire Line
+	4000 2000 4750 2000
+Wire Wire Line
+	4000 2100 4750 2100
+Connection ~ 4150 2200
+$Comp
+L GND #PWR?
+U 1 1 5F41102D
+P 4450 2300
+F 0 "#PWR?" H 4450 2050 50  0001 C CNN
+F 1 "GND" H 4450 2150 50  0000 C CNN
+F 2 "" H 4450 2300 50  0000 C CNN
+F 3 "" H 4450 2300 50  0000 C CNN
+	1    4450 2300
+	1    0    0    -1
+$EndComp
+Wire Wire Line
+	4750 2300 4450 2300
+Wire Wire Line
+	4000 4350 4750 4350
+Wire Wire Line
+	4000 4450 4750 4450
+Wire Wire Line
+	4000 4550 4750 4550
+Connection ~ 4250 4650
+$Comp
+L 7SEGMENTS AFF?
+U 1 1 5F411038
+P 7150 2400
+F 0 "AFF?" H 7150 2950 50  0000 C CNN
+F 1 "7SEGMENTS" H 7150 1950 50  0000 C CNN
+F 2 "" H 7150 2400 50  0000 C CNN
+F 3 "" H 7150 2400 50  0000 C CNN
+	1    7150 2400
+	1    0    0    -1
+$EndComp
+$Comp
+L 7SEGMENTS AFF?
+U 1 1 5F41103F
+P 7150 4750
+F 0 "AFF?" H 7150 5300 50  0000 C CNN
+F 1 "7SEGMENTS" H 7150 4300 50  0000 C CNN
+F 2 "" H 7150 4750 50  0000 C CNN
+F 3 "" H 7150 4750 50  0000 C CNN
+	1    7150 4750
+	1    0    0    -1
+$EndComp
+$Comp
+L R_PACK8 RP?
+U 1 1 5F411046
+P 6350 2350
+F 0 "RP?" H 6350 2800 50  0000 C CNN
+F 1 "1K" H 6350 1900 50  0000 C CNN
+F 2 "" H 6350 2350 50  0000 C CNN
+F 3 "" H 6350 2350 50  0000 C CNN
+	1    6350 2350
+	1    0    0    -1
+$EndComp
+$Comp
+L +5V #PWR?
+U 1 1 5F41104D
+P 7750 1750
+F 0 "#PWR?" H 7750 1600 50  0001 C CNN
+F 1 "+5V" H 7750 1890 50  0000 C CNN
+F 2 "" H 7750 1750 50  0000 C CNN
+F 3 "" H 7750 1750 50  0000 C CNN
+	1    7750 1750
+	1    0    0    -1
+$EndComp
+Wire Wire Line
+	7750 1750 7750 2050
+$Comp
+L R_PACK8 RP?
+U 1 1 5F411054
+P 6350 4700
+F 0 "RP?" H 6350 5150 50  0000 C CNN
+F 1 "1K" H 6350 4250 50  0000 C CNN
+F 2 "" H 6350 4700 50  0000 C CNN
+F 3 "" H 6350 4700 50  0000 C CNN
+	1    6350 4700
+	1    0    0    -1
+$EndComp
+Text HLabel 4150 2550 3    60   Output ~ 0
+HOUR_PULSE
+Text HLabel 2250 4350 0    60   Input ~ 0
+MINUTE_CLK
 $EndSCHEMATC

Commit message: hours section
Parts:
- gave numbers to parts that had none: 8
Changed lines of the file:
@@
 $EndDescr
 $Comp
-L 74LS90 U?
+L 74LS90 U11
 U 1 1 5F410FEF
 P 3250 4650
-F 0 "U?" H 3350 4650 50  0000 C CNN
+F 0 "U11" H 3350 4650 50  0000 C CNN
 F 1 "74LS90" H 3450 4450 50  0000 C CNN
 F 2 "" H 3250 4650 50  0000 C CNN
@@
 $EndComp
 $Comp
-L 74LS92 U?
+L 74LS92 U10
 U 1 1 5F410FF6
 P 3250 2300
-F 0 "U?" H 3350 2300 50  0000 C CNN
+F 0 "U10" H 3350 2300 50  0000 C CNN
 F 1 "74LS92" H 3450 2100 50  0000 C CNN
 F 2 "" H 3250 2300 50  0000 C CNN
@@
 $EndComp
 $Comp
-L GND #PWR?
+L GND #PWR16
 U 1 1 5F410FFD
 P 2550 5150
-F 0 "#PWR?" H 2550 4900 50  0001 C CNN
+F 0 "#PWR16" H 2550 4900 50  0001 C CNN
 F 1 "GND" H 2550 5000 50  0000 C CNN
 F 2 "" H 2550 5150 50  0000 C CNN
@@
 	2550 4600 2550 5150
 $Comp
-L GND #PWR?
+L GND #PWR15
 U 1 1 5F411004
 P 2550 2850
-F 0 "#PWR?" H 2550 2600 50  0001 C CNN
+F 0 "#PWR15" H 2550 2600 50  0001 C CNN
 F 1 "GND" H 2550 2700 50  0000 C CNN
 F 2 "" H 2550 2850 50  0000 C CNN
@@
 	4000 2200 4750 2200
 $Comp
-L 74LS47 U?
+L 74LS47 U12
 U 1 1 5F41101C
 P 5450 2350
-F 0 "U?" H 5450 2450 50  0000 C CNN
+F 0 "U12" H 5450 2450 50  0000 C CNN
 F 1 "74LS47" H 5450 2250 50  0000 C CNN
 F 2 "" H 5450 2350 50  0000 C CNN
@@
 $EndComp
 $Comp
-L 74LS47 U?
+L 74LS47 U13
 U 1 1 5F411023
 P 5450 4700
-F 0 "U?" H 5450 4800 50  0000 C CNN
+F 0 "U13" H 5450 4800 50  0000 C CNN
 F 1 "74LS47" H 5450 4600 50  0000 C CNN
 F 2 "" H 5450 4700 50  0000 C CNN
@@
 Connection ~ 4150 2200
 $Comp
-L GND #PWR?
+L GND #PWR17
 U 1 1 5F41102D
 P 4450 2300
-F 0 "#PWR?" H 4450 2050 50  0001 C CNN
+F 0 "#PWR17" H 4450 2050 50  0001 C CNN
 F 1 "GND" H 4450 2150 50  0000 C CNN
 F 2 "" H 4450 2300 50  0000 C CNN
@@
 Connection ~ 4250 4650
 $Comp
-L 7SEGMENTS AFF?
+L 7SEGMENTS AFF3
 U 1 1 5F411038
 P 7150 2400
-F 0 "AFF?" H 7150 2950 50  0000 C CNN
+F 0 "AFF3" H 7150 2950 50  0000 C CNN
 F 1 "7SEGMENTS" H 7150 1950 50  0000 C CNN
 F 2 "" H 7150 2400 50  0000 C CNN
@@
 $EndComp
 $Comp
-L 7SEGMENTS AFF?
+L 7SEGMENTS AFF4
 U 1 1 5F41103F
 P 7150 4750
-F 0 "AFF?" H 7150 5300 50  0000 C CNN
+F 0 "AFF4" H 7150 5300 50  0000 C CNN
 F 1 "7SEGMENTS" H 7150 4300 50  0000 C CNN
 F 2 "" H 7150 4750 50  0000 C CNN
@@
 $EndComp
 $Comp
-L R_PACK8 RP?
+L R_PACK8 RP3
 U 1 1 5F411046
 P 6350 2350
-F 0 "RP?" H 6350 2800 50  0000 C CNN
+F 0 "RP3" H 6350 2800 50  0000 C CNN
 F 1 "1K" H 6350 1900 50  0000 C CNN
 F 2 "" H 6350 2350 50  0000 C CNN
@@
 $EndComp
 $Comp
-L +5V #PWR?
+L +5V #PWR18
 U 1 1 5F41104D
 P 7750 1750
-F 0 "#PWR?" H 7750 1600 50  0001 C CNN
+F 0 "#PWR18" H 7750 1600 50  0001 C CNN
 F 1 "+5V" H 7750 1890 50  0000 C CNN
 F 2 "" H 7750 1750 50  0000 C CNN
@@
 	7750 1750 7750 2050
 $Comp
-L R_PACK8 RP?
+L R_PACK8 RP4
 U 1 1 5F411054
 P 6350 4700
-F 0 "RP?" H 6350 5150 50  0000 C CNN
+F 0 "RP4" H 6350 5150 50  0000 C CNN
 F 1 "1K" H 6350 4250 50  0000 C CNN
 F 2 "" H 6350 4700 50  0000 C CNN
