File: kicad/seconds.sch (KiCad schematic (older format))
At the start: 8 parts, among them U6 74LS92, U7 74LS90, U8 74LS47, U9 74LS47

Commit message: minute segment
Changed lines of the file:
@@
 Wire Wire Line
 	1800 2350 1800 2950
-Text GLabel 1500 4450 0    60   Input ~ 0
-SECOND_CLK
 Wire Wire Line
 	1800 4450 1500 4450
@@
 Wire Wire Line
 	1800 1800 1800 2200
-Text GLabel 3400 3350 1    60   Output ~ 0
-MINUTE_PULSE
 Wire Wire Line
 	3400 2650 3400 2300
@@
 	1    0    0    -1
 $EndComp
+Text HLabel 3400 2650 3    60   Output ~ 0
+MINUTE_PULSE
+Text HLabel 1500 4450 0    60   Input ~ 0
+SECOND_CLK
 $EndSCHEMATC

Commit message: hours section
Parts:
- gave numbers to parts that had none: 2
Changed lines of the file:
@@
 $EndComp
 $Comp
-L R_PACK8 RP?
+L R_PACK8 RP1
 U 1 1 5F40EE6E
 P 5600 2450
-F 0 "RP?" H 5600 2900 50  0000 C CNN
+F 0 "RP1" H 5600 2900 50  0000 C CNN
 F 1 "1K" H 5600 2000 50  0000 C CNN
 F 2 "" H 5600 2450 50  0000 C CNN
@@
 $EndComp
 $Comp
-L +5V #PWR?
+L +5V #PWR14
 U 1 1 5F40F2DD
 P 7000 1850
-F 0 "#PWR?" H 7000 1700 50  0001 C CNN
+F 0 "#PWR14" H 7000 1700 50  0001 C CNN
 F 1 "+5V" H 7000 1990 50  0000 C CNN
 F 2 "" H 7000 1850 50  0000 C CNN
@@
 	7000 1850 7000 2150
 $Comp
-L R_PACK8 RP?
+L R_PACK8 RP2
 U 1 1 5F40F321
 P 5600 4800
-F 0 "RP?" H 5600 5250 50  0000 C CNN
+F 0 "RP2" H 5600 5250 50  0000 C CNN
 F 1 "1K" H 5600 4350 50  0000 C CNN
 F 2 "" H 5600 4800 50  0000 C CNN
